Commit message: [update][chg][build_evn] 1. update catkin build install the project. 2. change the path of autolabor projects. [add][3d_slam_script] [fix][3d_slam] fix the bug in 3d slam with using cartographer.
Signed-off-by: wangqi <wangqi@shtdtech.com>

File: Autolabor/simulation/autolabor_description/urdf/autolabor_pro1_track_suit.urdf (robot description, URDF)
Before this commit: robot autolabor_description, 3 links, 2 joints
Links:
- removed link rslidar
- added link lidar_back; visual cylinder length=0.05 radius=0.03
- added link lidar_front; visual cylinder length=0.05 radius=0.03
Joints:
- added joint laser_back_link_joint: type fixed, parent base_link, child lidar_back, origin xyz=-0.4355 0.0 0.05 rpy=3.14 0.0 -3.14
