Commit message: [update][create_map] the first version for mapping use cartographer with rslidar-16
Signed-off-by: wangqi <wangqi@shtdtech.com>

File: Autolabor/simulation/autolabor_description/urdf/autolabor_pro1_track_suit_3d.urdf (robot description, URDF)
Before this commit: robot autolabor_description, 3 links, 2 joints
Joints:
- joint rslidar_link_joint: origin xyz=0.09 0.0 0.60 rpy=0.0 0.0 -3.14 -> xyz=0.09 0.0 0.60 rpy=0.0 0.0 3.1416

Commit message: [add][DGT001M]

File: Autolabor/simulation/autolabor_description/urdf/autolabor_pro1_track_suit_3d.urdf (robot description, URDF)
Before this commit: robot autolabor_description, 3 links, 2 joints
Joints:
- joint rslidar_link_joint: origin xyz=0.09 0.0 0.60 rpy=0.0 0.0 3.1416 -> xyz=0.004 0.0 0.60 rpy=0.0 0.0 0.0

Commit message: [update][cartographer][cartographer_ros][ceres-slover] 1.cartogragher version 2.0.0, Relevant Commits @ sides.pdf 2.cartogragher_ros version master 29 Jan commit 3.ceres-slover version 2.0.0 Signed-off-by: Imp <st.paul@foxmail.com>

File: Autolabor/simulation/autolabor_description/urdf/autolabor_pro1_track_suit_3d.urdf (robot description, URDF)
Before this commit: robot autolabor_description, 3 links, 2 joints
Links:
- link base_link: geometry collision box size=0.001 0.001 0.001; visual mesh filename=package://autolabor_description/meshes/autolabor_pro1.stl scale=0.001 0.001 0.001

Commit message: [update][navigation][teb_local_planner]
Signed-off-by: Imp <st.paul@foxmail.com>

File: Autolabor/simulation/autolabor_description/urdf/autolabor_pro1_track_suit_3d.urdf (robot description, URDF)
Before this commit: robot autolabor_description, 3 links, 2 joints
Links:
- added link base_footprint; collision box size=0.001 0.001 0.001; visual box size=0.001 0.001 0.001
Joints:
- added joint base_footprint_joint: type fixed, parent base_footprint, child base_link, origin xyz=0.0 0.0 0.14 rpy=0 0 0
- joint rslidar_link_joint: origin xyz=0.004 0.0 0.60 rpy=0.0 0.0 0.0 -> xyz=0.004 0.0 0.50 rpy=0.0 0.0 0.0

Commit message: [update][version1.0]
Signed-off-by: Imp <st.paul@foxmail.com>

File: Autolabor/simulation/autolabor_description/urdf/autolabor_pro1_track_suit_3d.urdf (robot description, URDF)
Before this commit: robot autolabor_description, 4 links, 3 joints
Joints:
- joint base_footprint_joint: origin xyz=0.0 0.0 0.14 rpy=0 0 0 -> xyz=0.0 0.0 0.6 rpy=0 0 0
